File: shichi-pcb.sch (KiCad schematic (older format))
At the start: 30 parts

Commit message: Assign PCB footprints to schematic symbols
Parts:
- C1, C2, C3, C4, C5, C6, C7, C8, C9: renamed from C?; footprint (none) -> Capacitor_SMD:C_0805_2012Metric_Pad1.15x1.40mm_HandSolder
- J1: renamed from J?; footprint (none) -> USB_Type-C:USB_C_Receptacle_HRO_TYPE-C-31-M-12-HandSoldering
- J10, J11, J2, J3, J4, J5, J6, J7, J8, J9: renamed from J?; footprint (none) -> Connector_PinHeader_2.54mm:PinHeader_1x01_P2.54mm_Vertical
- R1, R2, R3, R4, R5, R6: renamed from R?; footprint (none) -> Resistor_SMD:R_0805_2012Metric_Pad1.15x1.40mm_HandSolder
- SW1: renamed from SW?; footprint (none) -> Button_Switch_SMD:SW_SPST_TL3342
- Y1: renamed from Y?; footprint (none) -> Crystal:Crystal_SMD_SeikoEpson_FA238-4Pin_3.2x2.5mm_HandSoldering
- gave numbers to parts that had none: 2

Commit message: Use custom symbol for USB C Receptacle USB C Receptacle from 5.1.2 symbol library VBUS and GND are set to power input instead of power output
Parts:
- J1: value USB_C_Receptacle_USB2.0 -> USB_C_Receptacle_HRO_TYPE-C-31-M-12; symbol Connector:USB_C_Receptacle_USB2.0 -> USB_Type-C:USB_C_Receptacle_HRO_TYPE-C-31-M-12
Changed lines of the file:
@@
 $EndDescr
 $Comp
-L Connector:USB_C_Receptacle_USB2.0 J1
+L USB_Type-C:USB_C_Receptacle_HRO_TYPE-C-31-M-12 J1
 U 1 1 5CF95BEF
 P 1100 5800
 F 0 "J1" H 1207 6667 50  0000 C CNN
-F 1 "USB_C_Receptacle_USB2.0" H 1207 6576 50  0000 C CNN
+F 1 "USB_C_Receptacle_HRO_TYPE-C-31-M-12" H 1207 6576 50  0000 C CNN
 F 2 "USB_Type-C:USB_C_Receptacle_HRO_TYPE-C-31-M-12-HandSoldering" H 1250 5800 50  0001 C CNN
 F 3 "https://www.usb.org/sites/default/files/documents/usb_type-c.zip" H 1250 5800 50  0001 C CNN

Commit message: Fix XTAL1 ground short
Connections:
- net GND: no longer C1.2, U2.17 (XTAL1), Y1.1
- new net XTAL1: C1.2, U2.17 (XTAL1), Y1.1

Commit message: Use vertical group headers instead of individual headers
Parts:
- removed J10: RES, Connector_PinHeader_2.54mm:PinHeader_1x01_P2.54mm_Vertical, symbol Connector_Generic:Conn_01x01
- removed J11, J5: GND, Connector_PinHeader_2.54mm:PinHeader_1x01_P2.54mm_Vertical, symbol Connector_Generic:Conn_01x01
- removed J2, J7: VCC, Connector_PinHeader_2.54mm:PinHeader_1x01_P2.54mm_Vertical, symbol Connector_Generic:Conn_01x01
- removed J3: D-, Connector_PinHeader_2.54mm:PinHeader_1x01_P2.54mm_Vertical, symbol Connector_Generic:Conn_01x01
- removed J4: D+, Connector_PinHeader_2.54mm:PinHeader_1x01_P2.54mm_Vertical, symbol Connector_Generic:Conn_01x01
- removed J6: MISO, Connector_PinHeader_2.54mm:PinHeader_1x01_P2.54mm_Vertical, symbol Connector_Generic:Conn_01x01
- removed J8: SCK, Connector_PinHeader_2.54mm:PinHeader_1x01_P2.54mm_Vertical, symbol Connector_Generic:Conn_01x01
- removed J9: MOSI, Connector_PinHeader_2.54mm:PinHeader_1x01_P2.54mm_Vertical, symbol Connector_Generic:Conn_01x01
- added J2: Conn_01x04_Male, Connector_PinHeader_2.54mm:PinHeader_1x04_P2.54mm_Vertical, symbol Connector:Conn_01x04_Male
- added J3: Conn_01x06_Male, Connector_PinHeader_2.54mm:PinHeader_1x06_P2.54mm_Vertical, symbol Connector:Conn_01x06_Male
Connections:
- net GND: now also J2.4 (Pin_4), J3.6 (Pin_6)
- net MISO: now also J3.1 (Pin_1)
- net MOSI: now also J3.4 (Pin_4)
- net RESET: now also J3.5 (Pin_5)
- net SCK: now also J3.3 (Pin_3)
- net VCC: now also J2.1 (Pin_1), J3.2 (Pin_2)
- net at J1.A6 (D+), J1.B6 (D+), R4.1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: now also J2.3 (Pin_3)
- net at J1.A7 (D-), J1.B7 (D-), R3.1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: now also J2.2 (Pin_2)
Other:
- moved on the sheet: R3, R4

Commit message: Ground XTAL capacitors
Connections:
- net GND: now also C1.1, C2.2
Changed lines of the file:
@@
 Connection ~ 3000 5500
 Wire Wire Line
-	1650 3800 2350 3800
-Wire Wire Line
-	2000 3850 2000 3750
-Wire Wire Line
 	2000 3300 2000 3250
 Wire Wire Line
@@
 Wire Wire Line
 	1850 3750 2000 3750
-Connection ~ 2000 3750
-Wire Wire Line
-	2000 3750 2000 3700
 $Comp
 L power:VCC #PWR08
@@
 	3600 5900 3700 5900
 Wire Wire Line
+	2000 3850 2000 3800
+Wire Wire Line
+	2350 3800 2000 3800
+Connection ~ 2000 3800
+Wire Wire Line
+	1650 3800 2000 3800
+Wire Wire Line
 	5600 3200 6900 3200
 Wire Bus Line
@@
 Wire Bus Line
 	7500 2500 7500 6000
+Wire Wire Line
+	2000 3700 2000 3750
+Connection ~ 2000 3750
+Wire Wire Line
+	2000 3750 2000 3800
 $EndSCHEMATC
