File: shichi-pcb.kicad_pcb (KiCad board)
At the start: 2 copper layers, 266 x 96 mm, 176 parts, among them J1 USB_C_Receptacle_HRO_TYPE-C-3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, J2 Conn_01x04_Male, J3 Conn_01x06_Male, J4 Conn_01x04_Male, J5 Conn_01x02_Male, J6 Conn_01x01_Male, K1 SW_Push, K10 SW_Push, K11 SW_Push, K12 SW_Push, K13 SW_Push, K14 SW_Push, K15 SW_Push, K16 SW_Push, K17 SW_Push, K18 SW_Push, K19 SW_Push, K2 SW_Push, K20 SW_Push, K21 SW_Push, K22 SW_Push, K23 SW_Push, K24 SW_Push, K25 SW_Push, K26 SW_Push, K27 SW_Push, K28 SW_Push, K29 SW_Push, K3 SW_Push, K30 SW_Push, K31 SW_Push, K32 SW_Push, K33 SW_Push, K34 SW_Push, K35 SW_Push, K36 SW_Push, K37 SW_Push, K38 SW_Push, K39 SW_Push, K4 SW_Push, K40 SW_Push, K41 SW_Push, K42 SW_Push, K43 SW_Push, K44 SW_Push, K45 SW_Push, K46 SW_Push, K47 SW_Push, K48 SW_Push, K49 SW_Push, K5 SW_Push, K50 SW_Push, K51 SW_Push, K52 SW_Push, K53 SW_Push, K54 SW_Push, K55 SW_Push, K56 SW_Push, K57 SW_Push, K58 SW_Push, K59 SW_Push, K6 SW_Push, K60 SW_Push, K61 SW_Push, K62 SW_Push, K63 SW_Push, K64 SW_Push, K65 SW_Push, K66 SW_Push, K67 SW_Push, K68 SW_Push, K69 SW_Push, K7 SW_Push, K70 SW_Push, K71 SW_Push, K72 SW_Push, K8 SW_Push, K9 SW_Push, SW1 SW_Push, SW2 SW_Push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

Commit message: Add GND filled zone on F.CU and B.Cu
Routing:
- added copper zone on B.Cu, net GND
- added copper zone on F.Cu, net GND
Changed lines of the file:
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@@
   (segment (start 181.25 89.926998) (end 179.323002 88) (width 0.25) (layer B.Cu) (net 120))
   (segment (start 179.323002 88) (end 170.815 88) (width 0.25) (layer B.Cu) (net 120) (status 20))
+  (zone (net 1) (net_name GND) (layer F.Cu) (hatch edge 0.508)
+    (connect_pads (clearance 0.254))
+    (min_thickness 0.254)
+    (fill yes (arc_segments 32) (thermal_gap 0.508) (thermal_bridge_width 0.508))
+    (polygon
+      (pts
+        (xy 48.1 48.1) (xy 317.9 48.1) (xy 317.9 146.9) (xy 48.1 146.9)
+      )
+    )
+  )
+  (zone (net 1) (net_name GND) (layer B.Cu) (hatch edge 0.508)
+    (connect_pads (clearance 0.508))
+    (min_thickness 0.254)
+    (fill yes (arc_segments 32) (thermal_gap 0.508) (thermal_bridge_width 0.508))
+    (polygon
+      (pts
+        (xy 46.2 46.2) (xy 319.8 46.2) (xy 319.8 148.8) (xy 46.2 148.8)
+      )
+    )
+  )
 )
